Commit message: Initial commit with local modifications to SoftHand-Plugin

File: softhands_description/urdf/softhands.urdf.xacro (robot description, xacro)
@@ -38,10 +38,10 @@
 -->
 <robot name="softhand" xmlns:xacro="http://www.ros.org/wiki/xacro">
-  	<xacro:arg name="sh_version" default="v1_2_research"/>
+  	<xacro:arg name="sh_version" default="v3"/>
     <xacro:include filename="$(find softhands_description)/urdf/softhands.xacro"/>
     <xacro:softhands
         version="$(arg sh_version)"
         position="0 0 0"
-        orientation="0 0 0"
+        orientation="3.14 1.57 0"
         fixed_hands="false">
     </xacro:softhands>

File: softhands_description/urdf/softhands.xacro (robot description, xacro)
@@ -46,5 +46,5 @@
 		<xacro:include filename="$(find softhands_description)/urdf/xacro/include/macro/plugin.xacro"/>
 		<!-- If you are using only the hand -->
-		<link name="world"/>
+		<!-- <link name="world"/> -->
 		<!-- IF VERSION == 1_2_Research -->
 		<xacro:if value="${version == 'v1_2_research'}">
@@ -80,5 +80,5 @@
 				side="right"
 				parent="world"
-				position=" 0 0.2 0.02"
+				position="0 0.2 0.02"
 				orientation="${orientation}"
 				fixed_hands="false">
@@ -89,16 +89,16 @@
 			<xacro:include filename="$(find softhands_description)/urdf/xacro/include/macro/v3/header.xacro"/>
 			<xacro:include filename="$(find softhands_description)/urdf/xacro/v3.xacro"/>
-			<xacro:v3
+			<!-- <xacro:v3
 				side="left"
 				parent="world"
-				position="0.2 0 0.2"
-				orientation="1.57 0 3.14"
+				position="0 -0.2 0.02"
+				orientation="${orientation}"
 				fixed_hands="false">
-			</xacro:v3>
+			</xacro:v1_wide> -->
 			<xacro:v3
 				side="right"
-				parent="world"
-				position="0 0 0.2"
-				orientation="1.57 0 0"
+				parent="right_wrist"
+				position="0.015 -0.088 0.01"
+				orientation="${orientation}"
 				fixed_hands="false">
 			</xacro:v3>

File: softhands_description/urdf/xacro/include/macro/v3/modules/finger.xacro (robot description, xacro)
@@ -40,11 +40,15 @@
   <xacro:macro name="finger" params="yaml_file:=^ ns name parent side ">
     <!-- Knuckle -->
-    <xacro:phalanx_knuckle name="${name}" type="knuckle" parent="${parent}" ns="${ns}" side="${side}"/>
+    <xacro:phalanx_knuckle name="${name}" type="knuckle" parent="${parent}" ns="${ns}" side="${side}">
+    </xacro:phalanx_knuckle>
     <!-- Proximal -->
-    <xacro:phalanx_generic name="${name}" type="proximal" parent="${name}_knuckle" ns="${ns}" side="${side}"/>
+    <xacro:phalanx_generic name="${name}" type="proximal" parent="${name}_knuckle" ns="${ns}" side="${side}">
+    </xacro:phalanx_generic>
     <!-- Middle -->
-    <xacro:phalanx_generic name="${name}" type="middle" parent="${name}_proximal" ns="${ns}" side="${side}"/>
+    <xacro:phalanx_generic name="${name}" type="middle" parent="${name}_proximal" ns="${ns}" side="${side}">
+    </xacro:phalanx_generic>
     <!-- Distal -->
-    <xacro:phalanx_generic name="${name}" type="distal" parent="${name}_middle" ns="${ns}" side="${side}"/>
+    <xacro:phalanx_generic name="${name}" type="distal" parent="${name}_middle" ns="${ns}" side="${side}">
+    </xacro:phalanx_generic>
   </xacro:macro>
 </robot>

File: softhands_description/urdf/xacro/include/macro/v3/modules/palm/palm.xacro (robot description, xacro)
@@ -39,39 +39,33 @@
 <robot name="palm_v3" xmlns:xacro="http://www.ros.org/wiki/xacro">
 	<xacro:macro name="palm" params="ns name parent *origin">
-    <!-- Proximal JOINT -->
-    <joint name="${ns}_${name}_joint" type="fixed">
-      <xacro:insert_block name="origin"/>
-      <parent link="${parent}"/>
-      <child link="${ns}_${name}_link"/>
-      <axis xyz="0 0 -1"/>
-      <limit effort="30" velocity="10.0" lower="-0.524" upper="0.524" />
-      <dynamics damping="$(arg damping)" friction="$(arg friction)" />
-    </joint>
-    <!-- LINK -->
-    <link name="${ns}_${name}_link">
-        <inertial>
-          <mass value="${yaml_file[side][name]['mass']}"/>
-          <inertia ixx="${yaml_file[side][name]['inertia']['ixx']}" ixy="${yaml_file[side][name]['inertia']['ixy']}" ixz="${yaml_file[side][name]['inertia']['ixz']}" iyy="${yaml_file[side][name]['inertia']['iyy']}" iyz="${yaml_file[side][name]['inertia']['iyz']}" izz="${yaml_file[side][name]['inertia']['izz']}"/>
-          <origin rpy="0 0 0" xyz="${yaml_file[side][name]['inertia_origin']['position']}"/>
-        </inertial>
-      <visual>
-        <origin rpy="0 0 0" xyz="0 0 0"/>
-        <geometry>
-          <mesh filename="package://softhands_description/meshes/v3/${side}/${yaml_file[side][name]['mesh']}" scale="0.001 0.001 0.001"/>
-        </geometry>
-        <material name="qbhand/palm"/>
-      </visual>
-      <collision>
-        <origin rpy="0 0 0" xyz="0 0 0"/>
-        <geometry>
-          <mesh filename="package://softhands_description/meshes/v3/${side}/${yaml_file[side][name]['mesh_collision']}" scale="0.001 0.001 0.001"/>
-        </geometry>
-      </collision>
-    </link>
-        <!-- GAZEBO REF -->
-    <gazebo reference="${ns}_${name}_link">
-      <material>Gazebo/Grey</material>
-      <selfCollide>$(arg selfCollide)</selfCollide>
-    </gazebo>
+	  	<joint name="${ns}_palm_joint" type="fixed">
+			<xacro:insert_block name="origin"/>
+			<parent link="${parent}" />
+			<child link="${ns}_palm_link" />
+		</joint>
+		<link name="${ns}_palm_link">
+			<inertial>
+				<origin rpy="0 0 0" xyz="0.005 -4.037e-2 ${sign*1.214e-2}"/>
+				<mass value="2.27e-1"/>
+				<inertia ixx="1.14e-4" ixy="4.47e-6" ixz="-3.04e-6" iyy="7e-5" iyz="2.87e-6" izz="1.608e-4"/>
+			</inertial>
+			<visual>
+			<origin rpy="0 0 0" xyz="0 0 0"/>
+			<geometry>
+				<mesh filename="package://softhands_description/meshes/v3/${side}/palm_pinch.stl" scale="0.001 0.001 0.001"/>
+			</geometry>
+			<material name="qbhand/palm"/>
+			</visual>
+			<collision>
+				<origin rpy="0 0 0" xyz="0 0 0"/>
+				<geometry>
+					<mesh filename="package://softhands_description/meshes/v3/${side}/palm_pinch_collision.stl" scale="0.001 0.001 0.001"/>
+				</geometry>
+			</collision>
+		</link>
+		<gazebo reference="${ns}_palm_link">
+			<material>Gazebo/Grey</material>
+			<selfCollide>$(arg selfCollide)</selfCollide>
+		</gazebo>
 	</xacro:macro>
 </robot>

File: softhands_description/urdf/xacro/include/macro/v3/modules/thumb.xacro (robot description, xacro)
@@ -40,9 +40,12 @@
   <xacro:macro name="thumb" params="yaml_file:=^ ns name parent side">
     <!-- Knuckle -->
-    <xacro:thumb_knuckle name="${name}" type="knuckle" parent="${parent}" ns="${ns}" side="${side}"/>
+    <xacro:thumb_knuckle name="${name}" type="knuckle" parent="${parent}" ns="${ns}" side="${side}">
+    </xacro:thumb_knuckle>
     <!-- Proximal  -->
-    <xacro:phalanx_generic name="${name}" type="proximal" parent="${name}_knuckle" ns="${ns}" side="${side}"/>
+    <xacro:phalanx_generic name="${name}" type="proximal" parent="${name}_knuckle" ns="${ns}" side="${side}">
+    </xacro:phalanx_generic>
     <!--> Distal -->
-    <xacro:phalanx_generic name="${name}" type="distal" parent="${name}_proximal" ns="${ns}" side="${side}"/>
+    <xacro:phalanx_generic name="${name}" type="distal" parent="${name}_proximal" ns="${ns}" side="${side}">
+    </xacro:phalanx_generic>
   </xacro:macro>
 </robot>
